Commit message: init

File: src/cygnus_description/model/model.urdf (robot description, URDF)
Before this commit: robot Cygnus, 9 links, 8 joints
Links:
- link Cygnus__Aspa_1: geometry collision mesh filename=package://cygnus_description/meshes/aspa1.dae scale=0.01 0.01 0.01; visual mesh filename=package://cygnus_description/meshes/aspa1.dae scale=0.01 0.01 0.01
- link Cygnus__Aspa_2: geometry collision mesh filename=package://cygnus_description/meshes/aspa2.dae scale=0.01 0.01 0.01; visual mesh filename=package://cygnus_description/meshes/aspa2.dae scale=0.01 0.01 0.01
- link Cygnus__Aspa_3: geometry collision mesh filename=package://cygnus_description/meshes/aspa3_invert.dae scale=0.01 0.01 0.01; visual mesh filename=package://cygnus_description/meshes/aspa3_invert.dae scale=0.01 0.01 0.01
- link Cygnus__Aspa_4: geometry collision mesh filename=package://cygnus_description/meshes/aspa4_invert.dae scale=0.01 0.01 0.01; visual mesh filename=package://cygnus_description/meshes/aspa4_invert.dae scale=0.01 0.01 0.01
- link Cygnus__Cuerpo: geometry collision mesh filename=package://cygnus_description/meshes/Cuerpo.dae scale=0.01 0.01 0.01; visual mesh filename=package://cygnus_description/meshes/Cuerpo.dae scale=0.01 0.01 0.01
- link Cygnus__Motor_1: geometry collision mesh filename=package://cygnus_description/meshes/motor1.dae scale=0.01 0.01 0.01; visual mesh filename=package://cygnus_description/meshes/motor1.dae scale=0.01 0.01 0.01
- link Cygnus__Motor_2: geometry collision mesh filename=package://cygnus_description/meshes/motor2.dae scale=0.01 0.01 0.01; visual mesh filename=package://cygnus_description/meshes/motor2.dae scale=0.01 0.01 0.01
- link Cygnus__Motor_3: geometry collision mesh filename=package://cygnus_description/meshes/motor3.dae scale=0.01 0.01 0.01; visual mesh filename=package://cygnus_description/meshes/motor3.dae scale=0.01 0.01 0.01
- link Cygnus__Motor_4: geometry collision mesh filename=package://cygnus_description/meshes/motor4.dae scale=0.01 0.01 0.01; visual mesh filename=package://cygnus_description/meshes/motor4.dae scale=0.01 0.01 0.01
Joints:
- removed joint Cygnus__cuerpo_motor1
- removed joint Cygnus__cuerpo_motor2
- removed joint Cygnus__cuerpo_motor3
- removed joint Cygnus__cuerpo_motor4
- removed joint Cygnus__revo_motor1
- removed joint Cygnus__revo_motor2
- removed joint Cygnus__revo_motor3
- removed joint Cygnus__revo_motor4
- added joint Cygnus_cuerpo_motor1: type fixed, parent Cygnus__Cuerpo, child Cygnus__Motor_1, origin xyz=0.224874 -0.002     0.028 rpy=0  0  0, axis 0  0  0, limit lower=0 upper=0 effort=0 velocity=0
- added joint Cygnus_cuerpo_motor2: type fixed, parent Cygnus__Cuerpo, child Cygnus__Motor_2, origin xyz=-0.224874  0.002     0.028 rpy=0  0  0, axis 0  0  0, limit lower=0 upper=0 effort=0 velocity=0
- added joint Cygnus_cuerpo_motor3: type fixed, parent Cygnus__Cuerpo, child Cygnus__Motor_3, origin xyz=0.002     0.224874  0.028 rpy=0  0  0, axis 0  0  0, limit lower=0 upper=0 effort=0 velocity=0
- added joint Cygnus_cuerpo_motor4: type fixed, parent Cygnus__Cuerpo, child Cygnus__Motor_4, origin xyz=0.002    -0.224874  0.028 rpy=0  0  0, axis 0  0  0, limit lower=0 upper=0 effort=0 velocity=0
- added joint Cygnus_revo_motor1: type revolute, parent Cygnus__Motor_1, child Cygnus__Aspa_1, origin xyz=0.001   0.001   0.0315 rpy=0  0  0, axis 0  0  1, limit lower=0 upper=0 effort=0 velocity=50
- added joint Cygnus_revo_motor2: type revolute, parent Cygnus__Motor_2, child Cygnus__Aspa_2, origin xyz=-0.001799 -0.003     0.0315 rpy=0  0  0, axis 0  0  1, limit lower=0 upper=0 effort=0 velocity=50
- added joint Cygnus_revo_motor3: type revolute, parent Cygnus__Motor_3, child Cygnus__Aspa_3, origin xyz=-0.001799  0.002     0.0335 rpy=0  0  0, axis 0  0 -1, limit lower=0 upper=0 effort=0 velocity=50
- added joint Cygnus_revo_motor4: type revolute, parent Cygnus__Motor_4, child Cygnus__Aspa_4, origin xyz=-0.002   0.0024  0.0325 rpy=0  0  0, axis 0  0 -1, limit lower=0 upper=0 effort=0 velocity=50

Commit message: modify the joints references offset

File: src/cygnus_description/model/model.urdf (robot description, URDF)
Before this commit: robot Cygnus, 9 links, 8 joints
Links:
- removed link Cygnus__Cuerpo
- removed link Cygnus__Motor_1
- removed link Cygnus__Motor_2
- removed link Cygnus__Motor_3
- removed link Cygnus__Motor_4
- added link Cygnus_Cuerpo, mass 1.058; collision mesh filename=package://cygnus_description/meshes/Cuerpo.dae scale=0.01 0.01 0.01; visual mesh filename=package://cygnus_description/meshes/Cuerpo.dae scale=0.01 0.01 0.01
- added link Cygnus_Motor_1, mass 0.074; collision mesh filename=package://cygnus_description/meshes/motor1.dae scale=0.01 0.01 0.01; visual mesh filename=package://cygnus_description/meshes/motor1.dae scale=0.01 0.01 0.01
- added link Cygnus_Motor_2, mass 0.074; collision mesh filename=package://cygnus_description/meshes/motor2.dae scale=0.01 0.01 0.01; visual mesh filename=package://cygnus_description/meshes/motor2.dae scale=0.01 0.01 0.01
- added link Cygnus_Motor_3, mass 0.074; collision mesh filename=package://cygnus_description/meshes/motor3.dae scale=0.01 0.01 0.01; visual mesh filename=package://cygnus_description/meshes/motor3.dae scale=0.01 0.01 0.01
- added link Cygnus_Motor_4, mass 0.074; collision mesh filename=package://cygnus_description/meshes/motor4.dae scale=0.01 0.01 0.01; visual mesh filename=package://cygnus_description/meshes/motor4.dae scale=0.01 0.01 0.01
- added link base_link
Joints:
- added joint random_joint: type fixed, parent base_link, child Cygnus_Cuerpo, origin xyz=0 0 0 rpy=0  0  0, axis 0  0  0
- joint Cygnus_cuerpo_motor1: child Cygnus__Motor_1 -> Cygnus_Motor_1; origin xyz=0.224874 -0.002     0.028 rpy=0  0  0 -> xyz=0.224874 0 0.027 rpy=0  0  0; parent Cygnus__Cuerpo -> Cygnus_Cuerpo
- joint Cygnus_cuerpo_motor2: child Cygnus__Motor_2 -> Cygnus_Motor_2; origin xyz=-0.224874  0.002     0.028 rpy=0  0  0 -> xyz=-0.224874 0 0.027 rpy=0  0  0; parent Cygnus__Cuerpo -> Cygnus_Cuerpo
- joint Cygnus_cuerpo_motor3: child Cygnus__Motor_3 -> Cygnus_Motor_3; origin xyz=0.002     0.224874  0.028 rpy=0  0  0 -> xyz=0     0.224874  0.027 rpy=0  0  0; parent Cygnus__Cuerpo -> Cygnus_Cuerpo
- joint Cygnus_cuerpo_motor4: child Cygnus__Motor_4 -> Cygnus_Motor_4; origin xyz=0.002    -0.224874  0.028 rpy=0  0  0 -> xyz=0    -0.224874  0.027 rpy=0  0  0; parent Cygnus__Cuerpo -> Cygnus_Cuerpo
- joint Cygnus_revo_motor1: limit lower=0 upper=0 effort=0 velocity=50 -> effort=0.01428 velocity=254; origin xyz=0.001   0.001   0.0315 rpy=0  0  0 -> xyz=0 0 0.0055 rpy=0  0  0; parent Cygnus__Motor_1 -> Cygnus_Motor_1; type revolute -> continuous
- joint Cygnus_revo_motor2: limit lower=0 upper=0 effort=0 velocity=50 -> effort=0.01428 velocity=254; origin xyz=-0.001799 -0.003     0.0315 rpy=0  0  0 -> xyz=-0.004 0    0.0055 rpy=0  0  0; parent Cygnus__Motor_2 -> Cygnus_Motor_2; type revolute -> continuous
- joint Cygnus_revo_motor3: limit lower=0 upper=0 effort=0 velocity=50 -> effort=0.01428 velocity=254; origin xyz=-0.001799  0.002     0.0335 rpy=0  0  0 -> xyz=0  0    0 rpy=0  0  0; parent Cygnus__Motor_3 -> Cygnus_Motor_3; type revolute -> continuous
- joint Cygnus_revo_motor4: limit lower=0 upper=0 effort=0 velocity=50 -> effort=0.01428 velocity=254; origin xyz=-0.002   0.0024  0.0325 rpy=0  0  0 -> xyz=0   0  0 rpy=0  0  0; parent Cygnus__Motor_4 -> Cygnus_Motor_4; type revolute -> continuous
