Commit message: FEAT: propellers 3 and 4
propellers are set correctly in the URDF file

File: cygnus_description/model/model.urdf (robot description, URDF)
Before this commit: robot Cygnus, 6 links, 5 joints
Joints:
- joint Cygnus_revo_motor1: origin xyz=0 0 0 rpy=0  0  0 -> xyz=0.224 0 0.1 rpy=0  0  0
- joint Cygnus_revo_motor2: origin xyz=0 0 0 rpy=0  0  0 -> xyz=-0.224 0 0.1 rpy=0  0  0
- joint Cygnus_revo_motor3: origin xyz=0.0 0 0 rpy=0  0  0 -> xyz=0.0 0.224 0.062 rpy=0  0  0
- joint Cygnus_revo_motor4: origin xyz=0.0 0.0 0 rpy=0  0  0 -> xyz=0.0 -0.224 0.062 rpy=0  0  0

Commit message: FEAT: propellers 1 and 2

File: cygnus_description/model/model.urdf (robot description, URDF)
Before this commit: robot Cygnus, 6 links, 5 joints
Links:
- link Cygnus__Aspa_1: geometry collision cylinder length=0.006 radius=0.1; visual mesh filename=package://cygnus_description/meshes/aspa1.dae scale=0.01 0.01 0.01
- link Cygnus__Aspa_2: geometry collision cylinder length=0.006 radius=0.1; visual mesh filename=package://cygnus_description/meshes/aspa1.dae scale=0.01 0.01 0.01
Joints:
- joint Cygnus_revo_motor1: origin xyz=0.224 0 0.1 rpy=0  0  0 -> xyz=0.224 0 0.062 rpy=0  0  0
- joint Cygnus_revo_motor2: origin xyz=-0.224 0 0.1 rpy=0  0  0 -> xyz=-0.224 0 0.062 rpy=0  0  0

Commit message: FEAT: motor model
motor model attached to every propeller joint

File: cygnus_description/model/model.urdf (robot description, URDF)
Before this commit: robot Cygnus, 6 links, 5 joints
Joints:
- joint Cygnus_revo_motor2: axis 0  0  1 -> 0  0 -1; origin xyz=-0.224 0 0.062 rpy=0  0  0 -> xyz=0.0 -0.224 0.062 rpy=0  0  0
- joint Cygnus_revo_motor3: axis 0  0 -1 -> 0  0  1; origin xyz=0.0 0.224 0.062 rpy=0  0  0 -> xyz=-0.224 0 0.062 rpy=0  0  0
- joint Cygnus_revo_motor4: origin xyz=0.0 -0.224 0.062 rpy=0  0  0 -> xyz=0.0 0.224 0.062 rpy=0  0  0
