Commit message: REFACTOR: matching xml format

File: cygnus_description/model/cygnus.urdf (robot description, URDF)
Before this commit: robot cygnus, 6 links, 5 joints
Links:
- removed link Cygnus_Cuerpo
- removed link Cygnus__Aspa_1
- removed link Cygnus__Aspa_2
- removed link Cygnus__Aspa_3
- removed link Cygnus__Aspa_4
- added link cygnus_aspa_1, mass 0.007; collision cylinder length=0.006 radius=0.1; visual mesh filename=package://cygnus_description/meshes/aspa1.dae scale=0.01 0.01 0.01
- added link cygnus_aspa_2, mass 0.007; collision cylinder length=0.006 radius=0.1; visual mesh filename=package://cygnus_description/meshes/aspa1.dae scale=0.01 0.01 0.01
- added link cygnus_aspa_3, mass 0.007; collision cylinder length=0.006 radius=0.1; visual mesh filename=package://cygnus_description/meshes/aspa3_4.dae scale=1 1 1
- added link cygnus_aspa_4, mass 0.007; collision cylinder length=0.006 radius=0.1; visual mesh filename=package://cygnus_description/meshes/aspa3_4.dae scale=1 1 1
- added link cygnus_cuerpo, mass 1.3; collision box size=0.76 0.76 0.15; visual mesh filename=package://cygnus_description/meshes/cuerpo.dae scale=1 1 1
Joints:
- removed joint Cygnus_revo_motor1
- removed joint Cygnus_revo_motor2
- removed joint Cygnus_revo_motor3
- removed joint Cygnus_revo_motor4
- added joint cygnus_revo_motor_1: type continuous, parent base_link, child cygnus_aspa_1, origin xyz=0.224 0 0.062 rpy=0  0  0, axis 0  0  1, limit effort=0.01428 velocity=254
- added joint cygnus_revo_motor_2: type continuous, parent base_link, child cygnus_aspa_2, origin xyz=0.0 -0.224 0.062 rpy=0  0  0, axis 0  0 -1, limit effort=0.01428 velocity=254
- added joint cygnus_revo_motor_3: type continuous, parent base_link, child cygnus_aspa_3, origin xyz=-0.224 0 0.062 rpy=0  0  0, axis 0  0  1, limit effort=0.01428 velocity=254
- added joint cygnus_revo_motor_4: type continuous, parent base_link, child cygnus_aspa_4, origin xyz=0.0 0.224 0.062 rpy=0  0  0, axis 0  0 -1, limit effort=0.01428 velocity=254
- joint random_joint: child Cygnus_Cuerpo -> cygnus_cuerpo
